File: Hardware/Qwiic_Lidar_Lite/Production/Qwiic_Lidar_Lite-Panel.brd (EAGLE design)
At the start: 133.2 x 113.7 mm, 643 parts, among them U1 XC9140, U10 XC9140, U11 XC9140, U12 XC9140, U13 XC9140, U14 XC9140, U15 XC9140, U16 XC9140, U17 XC9140, U18 XC9140, U19 XC9140, U2 XC9140, U20 XC9140, U21 XC9140, U22 XC9140, U23 XC9140, U24 XC9140, U25 XC9140, U26 XC9140, U27 XC9140, U28 XC9140, U29 XC9140, U3 XC9140, U30 XC9140, U31 XC9140, U32 XC9140, U4 XC9140, U5 XC9140, U6 XC9140, U7 XC9140, U8 XC9140, U9 XC9140

Commit message: Updated board design with power LED
Parts:
- added D1, D10, D11, D12, D13, D14, D15, D16, D17, D18, D19, D2, D20, D21, D22, D23, D24, D25, D26, D27, D28, D29, D3, D30, D31, D32, D4, D5, D6, D7, D8, D9: RED, SparkFun-LED:LED-0603
- added R1, R10, R11, R12, R13, R14, R15, R16, R17, R18, R19, R2, R20, R21, R22, R23, R24, R25, R26, R27, R28, R29, R3, R30, R31, R32, R4, R5, R6, R7, R8, R9: 1k, SparkFun-Resistors:0603
- added U$353, U$365, U$377: (no value), buzzard_labels (2):GPIOB2
- added U$354, U$366, U$378: (no value), buzzard_labels (2):SCL1
- added U$355, U$367, U$379: (no value), buzzard_labels (2):SDA4
- added U$356, U$368, U$380: (no value), buzzard_labels (4):5V0
- added U$357, U$369, U$381: (no value), buzzard_labels (2):GPIOA5
- added U$358, U$370, U$382: (no value), buzzard_labels (5):QWIIC0
- added U$359, U$371, U$383: (no value), buzzard_labels (5):LIDAR#LITE1
- added U$360, U$372, U$384: (no value), buzzard_labels (6):PWR0
- added U$361, U$373: LIDAR_LITE, Qwiic_Lidar_Lite:LIDAR_LITE
- added U$362, U$374: (no value), buzzard_labels (2):GND3
- added U$363, U$375: (no value), buzzard_labels (2):3V30
- added U$364, U$376: SPARKX-LOGO4, SparkX:SPARKX-MEDIUM
- U$100, U$232: value LIDAR_LITE -> SPARKX-LOGO4; device Qwiic_Lidar_Lite:LIDAR_LITE -> SparkX:SPARKX-MEDIUM
- U$101, U$233: device buzzard_labels (2):GND3 -> buzzard_labels (2):GPIOB2
- U$102, U$234: device buzzard_labels (2):3V30 -> buzzard_labels (2):SCL1
- U$103, U$235: value SPARKX-LOGO4 -> (none); device SparkX:SPARKX-MEDIUM -> buzzard_labels (2):SDA4
- U$104, U$236: device buzzard_labels (2):GPIOB2 -> buzzard_labels (4):5V0
- U$105, U$237: device buzzard_labels (2):SCL1 -> buzzard_labels (2):GPIOA5
- U$106, U$238: device buzzard_labels (2):SDA4 -> buzzard_labels (5):QWIIC0
- U$107, U$239: device buzzard_labels (4):5V0 -> buzzard_labels (5):LIDAR#LITE1
- U$108, U$240: device buzzard_labels (2):GPIOA5 -> buzzard_labels (6):PWR0
- U$109, U$241: value (none) -> LIDAR_LITE; device buzzard_labels (5):QWIIC0 -> Qwiic_Lidar_Lite:LIDAR_LITE
- U$110, U$242: device buzzard_labels (5):LIDAR#LITE1 -> buzzard_labels (2):GND3
- U$111, U$243: value LIDAR_LITE -> (none); device Qwiic_Lidar_Lite:LIDAR_LITE -> buzzard_labels (2):3V30
- U$112, U$244: value (none) -> SPARKX-LOGO4; device buzzard_labels (2):GND3 -> SparkX:SPARKX-MEDIUM
- U$113, U$245: device buzzard_labels (2):3V30 -> buzzard_labels (2):GPIOB2
- U$114, U$246: value SPARKX-LOGO4 -> (none); device SparkX:SPARKX-MEDIUM -> buzzard_labels (2):SCL1
- U$115, U$247: device buzzard_labels (2):GPIOB2 -> buzzard_labels (2):SDA4
- U$116, U$248: device buzzard_labels (2):SCL1 -> buzzard_labels (4):5V0
- U$117, U$249: device buzzard_labels (2):SDA4 -> buzzard_labels (2):GPIOA5
- U$118, U$250: device buzzard_labels (4):5V0 -> buzzard_labels (5):QWIIC0
- U$119, U$251: device buzzard_labels (2):GPIOA5 -> buzzard_labels (5):LIDAR#LITE1
- U$12, U$144, U$276: value LIDAR_LITE -> (none); device Qwiic_Lidar_Lite:LIDAR_LITE -> buzzard_labels (6):PWR0
- U$120, U$252: device buzzard_labels (5):QWIIC0 -> buzzard_labels (6):PWR0
- U$121, U$253: value (none) -> LIDAR_LITE; device buzzard_labels (5):LIDAR#LITE1 -> Qwiic_Lidar_Lite:LIDAR_LITE
- U$122, U$254: value LIDAR_LITE -> (none); device Qwiic_Lidar_Lite:LIDAR_LITE -> buzzard_labels (2):GND3
- U$123, U$255: device buzzard_labels (2):GND3 -> buzzard_labels (2):3V30
- U$124, U$256: value (none) -> SPARKX-LOGO4; device buzzard_labels (2):3V30 -> SparkX:SPARKX-MEDIUM
- U$125, U$257: value SPARKX-LOGO4 -> (none); device SparkX:SPARKX-MEDIUM -> buzzard_labels (2):GPIOB2
- U$126, U$258: device buzzard_labels (2):GPIOB2 -> buzzard_labels (2):SCL1
- U$127, U$259: device buzzard_labels (2):SCL1 -> buzzard_labels (2):SDA4
- U$128, U$260: device buzzard_labels (2):SDA4 -> buzzard_labels (4):5V0
- U$129, U$261: device buzzard_labels (4):5V0 -> buzzard_labels (2):GPIOA5
- U$13, U$145, U$277: value (none) -> LIDAR_LITE; device buzzard_labels (2):GND3 -> Qwiic_Lidar_Lite:LIDAR_LITE
- U$130, U$262: device buzzard_labels (2):GPIOA5 -> buzzard_labels (5):QWIIC0
- U$131, U$263: device buzzard_labels (5):QWIIC0 -> buzzard_labels (5):LIDAR#LITE1
- U$132, U$264: device buzzard_labels (5):LIDAR#LITE1 -> buzzard_labels (6):PWR0
- U$14, U$146, U$278: device buzzard_labels (2):3V30 -> buzzard_labels (2):GND3
- U$147, U$15, U$279: value SPARKX-LOGO4 -> (none); device SparkX:SPARKX-MEDIUM -> buzzard_labels (2):3V30
- U$148, U$16, U$280: value (none) -> SPARKX-LOGO4; device buzzard_labels (2):GPIOB2 -> SparkX:SPARKX-MEDIUM
- U$149, U$17, U$281: device buzzard_labels (2):SCL1 -> buzzard_labels (2):GPIOB2
- U$150, U$18, U$282: device buzzard_labels (2):SDA4 -> buzzard_labels (2):SCL1
- U$151, U$19, U$283: device buzzard_labels (4):5V0 -> buzzard_labels (2):SDA4
- U$152, U$20, U$284: device buzzard_labels (2):GPIOA5 -> buzzard_labels (4):5V0
- U$153, U$21, U$285: device buzzard_labels (5):QWIIC0 -> buzzard_labels (2):GPIOA5
- U$154, U$22, U$286: device buzzard_labels (5):LIDAR#LITE1 -> buzzard_labels (5):QWIIC0
- U$155, U$23, U$287: value LIDAR_LITE -> (none); device Qwiic_Lidar_Lite:LIDAR_LITE -> buzzard_labels (5):LIDAR#LITE1
- U$156, U$24, U$288: device buzzard_labels (2):GND3 -> buzzard_labels (6):PWR0
- U$157, U$25, U$289: value (none) -> LIDAR_LITE; device buzzard_labels (2):3V30 -> Qwiic_Lidar_Lite:LIDAR_LITE
- U$158, U$26, U$290: value SPARKX-LOGO4 -> (none); device SparkX:SPARKX-MEDIUM -> buzzard_labels (2):GND3
- U$159, U$27, U$291: device buzzard_labels (2):GPIOB2 -> buzzard_labels (2):3V30
- U$160, U$28, U$292: value (none) -> SPARKX-LOGO4; device buzzard_labels (2):SCL1 -> SparkX:SPARKX-MEDIUM
- U$161, U$29, U$293: device buzzard_labels (2):SDA4 -> buzzard_labels (2):GPIOB2
- U$162, U$294, U$30: device buzzard_labels (4):5V0 -> buzzard_labels (2):SCL1
- U$163, U$295, U$31: device buzzard_labels (2):GPIOA5 -> buzzard_labels (2):SDA4
- U$164, U$296, U$32: device buzzard_labels (5):QWIIC0 -> buzzard_labels (4):5V0
- U$165, U$297, U$33: device buzzard_labels (5):LIDAR#LITE1 -> buzzard_labels (2):GPIOA5
- U$166, U$298, U$34: value LIDAR_LITE -> (none); device Qwiic_Lidar_Lite:LIDAR_LITE -> buzzard_labels (5):QWIIC0
- U$167, U$299, U$35: device buzzard_labels (2):GND3 -> buzzard_labels (5):LIDAR#LITE1
- U$168, U$300, U$36: device buzzard_labels (2):3V30 -> buzzard_labels (6):PWR0
- U$169, U$301, U$37: value SPARKX-LOGO4 -> LIDAR_LITE; device SparkX:SPARKX-MEDIUM -> Qwiic_Lidar_Lite:LIDAR_LITE
- U$170, U$302, U$38: device buzzard_labels (2):GPIOB2 -> buzzard_labels (2):GND3
- U$171, U$303, U$39: device buzzard_labels (2):SCL1 -> buzzard_labels (2):3V30
- U$172, U$304, U$40: value (none) -> SPARKX-LOGO4; device buzzard_labels (2):SDA4 -> SparkX:SPARKX-MEDIUM
- U$173, U$305, U$41: device buzzard_labels (4):5V0 -> buzzard_labels (2):GPIOB2
- U$174, U$306, U$42: device buzzard_labels (2):GPIOA5 -> buzzard_labels (2):SCL1
- U$175, U$307, U$43: device buzzard_labels (5):QWIIC0 -> buzzard_labels (2):SDA4
- U$176, U$308, U$44: device buzzard_labels (5):LIDAR#LITE1 -> buzzard_labels (4):5V0
- U$177, U$309, U$45: value LIDAR_LITE -> (none); device Qwiic_Lidar_Lite:LIDAR_LITE -> buzzard_labels (2):GPIOA5
- U$178, U$310, U$46: device buzzard_labels (2):GND3 -> buzzard_labels (5):QWIIC0
- U$179, U$311, U$47: device buzzard_labels (2):3V30 -> buzzard_labels (5):LIDAR#LITE1
- U$180, U$312, U$48: value SPARKX-LOGO4 -> (none); device SparkX:SPARKX-MEDIUM -> buzzard_labels (6):PWR0
- U$181, U$313, U$49: value (none) -> LIDAR_LITE; device buzzard_labels (2):GPIOB2 -> Qwiic_Lidar_Lite:LIDAR_LITE
- U$182, U$314, U$50: device buzzard_labels (2):SCL1 -> buzzard_labels (2):GND3
- U$183, U$315, U$51: device buzzard_labels (2):SDA4 -> buzzard_labels (2):3V30
- U$184, U$316, U$52: value (none) -> SPARKX-LOGO4; device buzzard_labels (4):5V0 -> SparkX:SPARKX-MEDIUM
- U$185, U$317, U$53: device buzzard_labels (2):GPIOA5 -> buzzard_labels (2):GPIOB2
- U$186, U$318, U$54: device buzzard_labels (5):QWIIC0 -> buzzard_labels (2):SCL1
- U$187, U$319, U$55: device buzzard_labels (5):LIDAR#LITE1 -> buzzard_labels (2):SDA4
- U$188, U$320, U$56: value LIDAR_LITE -> (none); device Qwiic_Lidar_Lite:LIDAR_LITE -> buzzard_labels (4):5V0
- U$189, U$321, U$57: device buzzard_labels (2):GND3 -> buzzard_labels (2):GPIOA5
- U$190, U$322, U$58: device buzzard_labels (2):3V30 -> buzzard_labels (5):QWIIC0
- U$191, U$323, U$59: value SPARKX-LOGO4 -> (none); device SparkX:SPARKX-MEDIUM -> buzzard_labels (5):LIDAR#LITE1
- U$192, U$324, U$60: device buzzard_labels (2):GPIOB2 -> buzzard_labels (6):PWR0
- U$193, U$325, U$61: value (none) -> LIDAR_LITE; device buzzard_labels (2):SCL1 -> Qwiic_Lidar_Lite:LIDAR_LITE
- U$194, U$326, U$62: device buzzard_labels (2):SDA4 -> buzzard_labels (2):GND3
- U$195, U$327, U$63: device buzzard_labels (4):5V0 -> buzzard_labels (2):3V30
- U$196, U$328, U$64: value (none) -> SPARKX-LOGO4; device buzzard_labels (2):GPIOA5 -> SparkX:SPARKX-MEDIUM
- U$197, U$329, U$65: device buzzard_labels (5):QWIIC0 -> buzzard_labels (2):GPIOB2
- U$198, U$330, U$66: device buzzard_labels (5):LIDAR#LITE1 -> buzzard_labels (2):SCL1
- U$199, U$331, U$67: value LIDAR_LITE -> (none); device Qwiic_Lidar_Lite:LIDAR_LITE -> buzzard_labels (2):SDA4
- U$200, U$332, U$68: device buzzard_labels (2):GND3 -> buzzard_labels (4):5V0
- U$201, U$333, U$69: device buzzard_labels (2):3V30 -> buzzard_labels (2):GPIOA5
- U$202, U$334, U$70: value SPARKX-LOGO4 -> (none); device SparkX:SPARKX-MEDIUM -> buzzard_labels (5):QWIIC0
- U$203, U$335, U$71: device buzzard_labels (2):GPIOB2 -> buzzard_labels (5):LIDAR#LITE1
- U$204, U$336, U$72: device buzzard_labels (2):SCL1 -> buzzard_labels (6):PWR0
- U$205, U$337, U$73: value (none) -> LIDAR_LITE; device buzzard_labels (2):SDA4 -> Qwiic_Lidar_Lite:LIDAR_LITE
- U$206, U$338, U$74: device buzzard_labels (4):5V0 -> buzzard_labels (2):GND3
- U$207, U$339, U$75: device buzzard_labels (2):GPIOA5 -> buzzard_labels (2):3V30
- U$208, U$340, U$76: value (none) -> SPARKX-LOGO4; device buzzard_labels (5):QWIIC0 -> SparkX:SPARKX-MEDIUM
- U$209, U$341, U$77: device buzzard_labels (5):LIDAR#LITE1 -> buzzard_labels (2):GPIOB2
- U$210, U$342, U$78: value LIDAR_LITE -> (none); device Qwiic_Lidar_Lite:LIDAR_LITE -> buzzard_labels (2):SCL1
- U$211, U$343, U$79: device buzzard_labels (2):GND3 -> buzzard_labels (2):SDA4
- U$212, U$344, U$80: device buzzard_labels (2):3V30 -> buzzard_labels (4):5V0
- U$213, U$345, U$81: value SPARKX-LOGO4 -> (none); device SparkX:SPARKX-MEDIUM -> buzzard_labels (2):GPIOA5
- U$214, U$346, U$82: device buzzard_labels (2):GPIOB2 -> buzzard_labels (5):QWIIC0
- U$215, U$347, U$83: device buzzard_labels (2):SCL1 -> buzzard_labels (5):LIDAR#LITE1
- U$216, U$348, U$84: device buzzard_labels (2):SDA4 -> buzzard_labels (6):PWR0
- U$217, U$349, U$85: value (none) -> LIDAR_LITE; device buzzard_labels (4):5V0 -> Qwiic_Lidar_Lite:LIDAR_LITE
- U$218, U$350, U$86: device buzzard_labels (2):GPIOA5 -> buzzard_labels (2):GND3
- U$219, U$351, U$87: device buzzard_labels (5):QWIIC0 -> buzzard_labels (2):3V30
- U$220, U$352, U$88: value (none) -> SPARKX-LOGO4; device buzzard_labels (5):LIDAR#LITE1 -> SparkX:SPARKX-MEDIUM
- U$221, U$89: value LIDAR_LITE -> (none); device Qwiic_Lidar_Lite:LIDAR_LITE -> buzzard_labels (2):GPIOB2
- U$222, U$90: device buzzard_labels (2):GND3 -> buzzard_labels (2):SCL1
- U$223, U$91: device buzzard_labels (2):3V30 -> buzzard_labels (2):SDA4
- U$224, U$92: value SPARKX-LOGO4 -> (none); device SparkX:SPARKX-MEDIUM -> buzzard_labels (4):5V0
- U$225, U$93: device buzzard_labels (2):GPIOB2 -> buzzard_labels (2):GPIOA5
- U$226, U$94: device buzzard_labels (2):SCL1 -> buzzard_labels (5):QWIIC0
- U$227, U$95: device buzzard_labels (2):SDA4 -> buzzard_labels (5):LIDAR#LITE1
- U$228, U$96: device buzzard_labels (4):5V0 -> buzzard_labels (6):PWR0
- U$229, U$97: value (none) -> LIDAR_LITE; device buzzard_labels (2):GPIOA5 -> Qwiic_Lidar_Lite:LIDAR_LITE
- U$230, U$98: device buzzard_labels (5):QWIIC0 -> buzzard_labels (2):GND3
- U$231, U$99: device buzzard_labels (5):LIDAR#LITE1 -> buzzard_labels (2):3V30
- moved U$89 131.1 mm to (105.4, 7.80)
- moved U$177 117.8 mm to (91.0, 28.8)
- moved U$188 117.2 mm to (107.7, 44.0)
- moved U$96 112.9 mm to (112.6, 1.07), flipped to the top
- moved U$186 112.4 mm to (106.9, 33.9)
- moved U$276 112.3 mm to (98.4, 48.2), flipped to the top
- moved U$187 112.0 mm to (106.6, 36.4)
- moved U$184 108.3 mm to (107.9, 25.4)
- moved U$90 104.6 mm to (106.9, 10.3)
- moved U$91 102.8 mm to (106.6, 12.9)
- moved U$93 102.7 mm to (105.3, 5.26)
- moved U$185 101.7 mm to (105.4, 31.3)
- moved U$183 101.6 mm to (106.6, 39.0)
- moved U$182 100.3 mm to (106.5, 41.5)
- moved U$92 99.3 mm to (107.7, 20.5)
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Connections:
- new net N$1: D1.A, R1.1
- new net N$10: D5.A, R5.1
- new net N$12: D6.A, R6.1
- new net N$14: D7.A, R7.1
- new net N$16: D8.A, R8.1
- new net N$18: D9.A, R9.1
- new net N$20: D10.A, R10.1
- new net N$22: D11.A, R11.1
- new net N$24: D12.A, R12.1
- new net N$26: D13.A, R13.1
- new net N$28: D14.A, R14.1
- new net N$30: D15.A, R15.1
- new net N$32: D16.A, R16.1
- new net N$34: D17.A, R17.1
- new net N$36: D18.A, R18.1
- new net N$38: D19.A, R19.1
- new net N$4: D2.A, R2.1
- new net N$40: D20.A, R20.1
- new net N$42: D21.A, R21.1
- new net N$44: D22.A, R22.1
- new net N$46: D23.A, R23.1
- new net N$48: D24.A, R24.1
- new net N$50: D25.A, R25.1
- new net N$52: D26.A, R26.1
- new net N$54: D27.A, R27.1
- new net N$56: D28.A, R28.1
- new net N$58: D29.A, R29.1
- new net N$6: D3.A, R3.1
- new net N$60: D30.A, R30.1
- new net N$62: D31.A, R31.1
- new net N$64: D32.A, R32.1
- new net N$8: D4.A, R4.1
- net 3.3V: now also R1.2
- net 3.3V1: now also R2.2
- net 3.3V10: now also R11.2
- net 3.3V11: now also R12.2
- net 3.3V12: now also R13.2
- net 3.3V13: now also R14.2
- net 3.3V14: now also R15.2
- net 3.3V15: now also R16.2
- net 3.3V16: now also R17.2
- net 3.3V17: now also R18.2
- net 3.3V18: now also R19.2
- net 3.3V19: now also R20.2
- net 3.3V2: now also R3.2
- net 3.3V20: now also R21.2
- net 3.3V21: now also R22.2
- net 3.3V22: now also R23.2
- net 3.3V23: now also R24.2
- net 3.3V24: now also R25.2
- net 3.3V25: now also R26.2
- net 3.3V26: now also R27.2
- net 3.3V27: now also R28.2
- net 3.3V28: now also R29.2
- net 3.3V29: now also R30.2
- net 3.3V3: now also R4.2
- net 3.3V30: now also R31.2
- net 3.3V31: now also R32.2
- net 3.3V4: now also R5.2
- net 3.3V5: now also R6.2
- net 3.3V6: now also R7.2
- net 3.3V7: now also R8.2
- net 3.3V8: now also R9.2
- net 3.3V9: now also R10.2
- net GND: now also D1.C
- net GND1: now also D2.C
- net GND10: now also D11.C
- net GND11: now also D12.C
- net GND12: now also D13.C
- net GND13: now also D14.C
- net GND14: now also D15.C
- net GND15: now also D16.C
- net GND16: now also D17.C
- net GND17: now also D18.C
- net GND18: now also D19.C
- net GND19: now also D20.C
- net GND2: now also D3.C
- net GND20: now also D21.C
- net GND21: now also D22.C
- net GND22: now also D23.C
- net GND23: now also D24.C
- net GND24: now also D25.C
- net GND25: now also D26.C
- net GND26: now also D27.C
- net GND27: now also D28.C
- net GND28: now also D29.C
- net GND29: now also D30.C
- net GND3: now also D4.C
- net GND30: now also D31.C
- net GND31: now also D32.C
- net GND4: now also D5.C
- net GND5: now also D6.C
- net GND6: now also D7.C
- net GND7: now also D8.C
- net GND8: now also D9.C
- net GND9: now also D10.C
Routing:
- net 3.3V6: track 29.6 -> 37.2 mm, vias 3 -> 5
- net 3.3V30: track 29.6 -> 37.2 mm, vias 3 -> 5
- net 3.3V14: track 29.6 -> 37.2 mm, vias 3 -> 5
- net 3.3V12: track 29.6 -> 37.2 mm, vias 3 -> 5
- net 3.3V22: track 29.6 -> 37.2 mm, vias 3 -> 5
- net 3.3V20: track 29.6 -> 37.2 mm, vias 3 -> 5
- net 3.3V18: track 29.6 -> 37.2 mm, vias 3 -> 5
- net 3.3V8: track 29.6 -> 37.2 mm, vias 3 -> 5
- net 3.3V4: track 29.6 -> 37.2 mm, vias 3 -> 5
- net 3.3V28: track 29.6 -> 37.2 mm, vias 3 -> 5
- net 3.3V2: track 29.6 -> 37.2 mm, vias 3 -> 5
- net 3.3V10: track 29.6 -> 37.2 mm, vias 3 -> 5
- net 3.3V26: track 29.6 -> 37.2 mm, vias 3 -> 5
- net 3.3V24: track 29.6 -> 37.2 mm, vias 3 -> 5
- net 3.3V16: track 29.6 -> 37.2 mm, vias 3 -> 5
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